File: Hardware/IMUnav_H00/IMUnav_H00.kicad_pcb (KiCad board)
At the start: 4 copper layers, 0 parts

Commit message: Added signal connections to MCU+misc
Parts:
- added BT1: Li-Ion 18650, Battery:BatteryHolder_MPD_BH-18650-PC2, F.Cu at (48.8, 36.2)
- added C1: 100n, Capacitor_SMD:C_0603_1608Metric, F.Cu at (122.1, 97.8)
- added C10: 2u2, Capacitor_SMD:C_0603_1608Metric, F.Cu at (126.1, 105.3)
- added C11: 2u2, Capacitor_SMD:C_0603_1608Metric, F.Cu at (126.1, 107.8)
- added C12: 100n, Capacitor_SMD:C_0603_1608Metric, F.Cu at (126.1, 110.3)
- added C13: 1u, Capacitor_SMD:C_0603_1608Metric, F.Cu at (47.1, 48.3)
- added C14: 100n, Capacitor_SMD:C_0603_1608Metric, F.Cu at (47.1, 50.8)
- added C15: 100n, Capacitor_SMD:C_0603_1608Metric, F.Cu at (47.1, 53.3)
- added C16: 4u7, Capacitor_SMD:C_0603_1608Metric, F.Cu at (47.1, 55.8)
- added C17: 4u7, Capacitor_SMD:C_0603_1608Metric, F.Cu at (47.1, 58.3)
- added C18: 100n, Capacitor_SMD:C_0603_1608Metric, F.Cu at (47.1, 60.8)
- added C19: 1u, Capacitor_SMD:C_0603_1608Metric, F.Cu at (47.1, 63.3)
- added C2: 100n, Capacitor_SMD:C_0603_1608Metric, F.Cu at (122.1, 100.3)
- added C20: 4u7, Capacitor_SMD:C_0603_1608Metric, F.Cu at (47.1, 65.8)
- added C21: 100n, Capacitor_SMD:C_0603_1608Metric, F.Cu at (47.1, 68.4)
- added C22: 4u7, Capacitor_SMD:C_0603_1608Metric, F.Cu at (47.1, 70.9)
- added C23: 1u, Capacitor_SMD:C_0603_1608Metric, F.Cu at (51.1, 48.3)
- added C24: 4u7, Capacitor_SMD:C_0603_1608Metric, F.Cu at (51.1, 50.8)
- added C25: 10n, Capacitor_SMD:C_0603_1608Metric, F.Cu at (51.1, 53.3)
- added C26: 10n, Capacitor_SMD:C_0603_1608Metric, F.Cu at (51.1, 55.8)
- added C27: 100n, Capacitor_SMD:C_0603_1608Metric, F.Cu at (51.1, 58.3)
- added C28: 10n, Capacitor_SMD:C_0603_1608Metric, F.Cu at (51.1, 60.8)
- added C29: 100n, Capacitor_SMD:C_0603_1608Metric, F.Cu at (51.1, 63.3)
- added C3: 100n, Capacitor_SMD:C_0603_1608Metric, F.Cu at (122.1, 102.8)
- added C30: 10n, Capacitor_SMD:C_0603_1608Metric, F.Cu at (51.1, 65.8)
- added C31: 1n, Capacitor_SMD:C_0402_1005Metric, F.Cu at (103.4, 70.5)
- added C32: 22u, Capacitor_SMD:C_0603_1608Metric, F.Cu at (51.1, 68.4)
- added C33: 22u, Capacitor_SMD:C_0603_1608Metric, F.Cu at (51.1, 70.9)
- added C34: 100n, Capacitor_SMD:C_0603_1608Metric, F.Cu at (55.1, 48.3)
- added C35: 22u, Capacitor_SMD:C_0603_1608Metric, F.Cu at (55.1, 50.8)
- added C36: 100n, Capacitor_SMD:C_0603_1608Metric, F.Cu at (55.1, 53.3)
- added C37: 10u, Capacitor_SMD:C_0603_1608Metric, F.Cu at (140.2, 118.9)
- added C38: 100n, Capacitor_SMD:C_0603_1608Metric, F.Cu at (140.2, 121.4)
- added C39: 100n, Capacitor_SMD:C_0603_1608Metric, F.Cu at (140.2, 123.9)
- added C4: 100n, Capacitor_SMD:C_0603_1608Metric, F.Cu at (122.1, 105.3)
- added C40: 1u, Capacitor_SMD:C_0603_1608Metric, F.Cu at (140.2, 126.4)
- added C41: 10u, Capacitor_SMD:C_0805_2012Metric, F.Cu at (160.0, 119.5)
- added C42: 10u, Capacitor_SMD:C_0805_2012Metric, F.Cu at (82.9, 116.3)
- added C43: 100n, Capacitor_SMD:C_0603_1608Metric, F.Cu at (66.6, 109.8)
- added C44: 100n, Capacitor_SMD:C_0603_1608Metric, F.Cu at (66.6, 112.3)
- added C45: 100n, Capacitor_SMD:C_0603_1608Metric, F.Cu at (66.6, 114.8)
- added C46: 100n, Capacitor_SMD:C_0603_1608Metric, F.Cu at (66.6, 117.3)
- added C47: 100n, Capacitor_SMD:C_0603_1608Metric, F.Cu at (66.6, 119.8)
- added C48: 2n2, Capacitor_SMD:C_0603_1608Metric, F.Cu at (66.6, 122.3)
- added C49: 100n, Capacitor_SMD:C_0603_1608Metric, F.Cu at (70.7, 109.8)
- added C5: 100n, Capacitor_SMD:C_0603_1608Metric, F.Cu at (122.1, 107.8)
- added C50: 100n, Capacitor_SMD:C_0603_1608Metric, F.Cu at (70.7, 112.3)
- added C51: 100n, Capacitor_SMD:C_0603_1608Metric, F.Cu at (70.7, 114.8)
- added C52: 10u, Capacitor_SMD:C_0805_2012Metric, F.Cu at (82.9, 119.4)
- added C53: 100n, Capacitor_SMD:C_0603_1608Metric, F.Cu at (70.7, 117.3)
- added C54: 100n, Capacitor_SMD:C_0603_1608Metric, F.Cu at (70.7, 119.8)
- added C55: 100n, Capacitor_SMD:C_0603_1608Metric, F.Cu at (70.7, 122.3)
- added C56: 100n, Capacitor_SMD:C_0603_1608Metric, F.Cu at (74.7, 109.8)
- added C57: 100n, Capacitor_SMD:C_0603_1608Metric, F.Cu at (74.7, 112.3)
- added C58: 100n, Capacitor_SMD:C_0603_1608Metric, F.Cu at (74.7, 114.8)
- added C59: 1u, Capacitor_SMD:C_0603_1608Metric, F.Cu at (140.2, 75.4)
- added C6: 100n, Capacitor_SMD:C_0603_1608Metric, F.Cu at (122.1, 110.3)
- added C60: 1u, Capacitor_SMD:C_0603_1608Metric, F.Cu at (140.2, 77.9)
- added C61: 100n, Capacitor_SMD:C_0603_1608Metric, F.Cu at (140.2, 80.4)
- added C62: 10u, Capacitor_SMD:C_0805_2012Metric, F.Cu at (159.7, 93.0)
- added C63: 100n, Capacitor_SMD:C_0603_1608Metric, F.Cu at (140.2, 82.9)
- added C64: 10u, Capacitor_SMD:C_0805_2012Metric, F.Cu at (159.7, 96.0)
- added C65: 100n, Capacitor_SMD:C_0603_1608Metric, F.Cu at (107.8, 118.3)
- added C66: 100n, Capacitor_SMD:C_0603_1608Metric, F.Cu at (107.8, 120.8)
- added C67: 100n, Capacitor_SMD:C_0603_1608Metric, F.Cu at (107.8, 123.3)
- added C68: 100n, Capacitor_SMD:C_0603_1608Metric, F.Cu at (167.6, 26.7)
- added C69: 100n, Capacitor_SMD:C_0603_1608Metric, F.Cu at (167.6, 29.2)
- added C7: 100n, Capacitor_SMD:C_0603_1608Metric, F.Cu at (126.1, 97.8)
- added C70: 100n, Capacitor_SMD:C_0603_1608Metric, F.Cu at (167.6, 31.8)
- added C71: 100n, Capacitor_SMD:C_0603_1608Metric, F.Cu at (167.6, 34.3)
- added C72: 100n, Capacitor_SMD:C_0603_1608Metric, F.Cu at (167.6, 36.8)
- added C8: 100n, Capacitor_SMD:C_0603_1608Metric, F.Cu at (126.1, 100.3)
- added C9: 100n, Capacitor_SMD:C_0603_1608Metric, F.Cu at (126.1, 102.8)
- added D1: LED_GREEN, LED_SMD:LED_0603_1608Metric, F.Cu at (87.3, 48.3)
- added D2: LED_RED, LED_SMD:LED_0603_1608Metric, F.Cu at (87.3, 50.9)
- added D3: LED_RED, LED_SMD:LED_0603_1608Metric, F.Cu at (87.3, 53.5)
- added D4: LED_GREEN, LED_SMD:LED_0603_1608Metric, F.Cu at (87.3, 56.1)
- added D5: B5819W, Diode_SMD:D_SOD-123, F.Cu at (104.9, 48.7)
- added D6: LED_YELLOW, LED_SMD:LED_0603_1608Metric, F.Cu at (139.1, 55.1)
- added D7: LED_YELLOW, LED_SMD:LED_0603_1608Metric, F.Cu at (139.1, 57.6)
- added D8: LED_YELLOW, LED_SMD:LED_0603_1608Metric, F.Cu at (139.1, 60.2)
- added FB1: GZ2012D101TF, Resistor_SMD:R_0805_2012Metric, F.Cu at (91.5, 48.5)
- added FB2: GZ2012D101TF, Resistor_SMD:R_0805_2012Metric, F.Cu at (91.5, 51.5)
- added FB3: GZ2012D101TF, Resistor_SMD:R_0805_2012Metric, F.Cu at (91.5, 54.4)
- added FB4: GZ2012D101TF, Resistor_SMD:R_0805_2012Metric, F.Cu at (144.4, 93.2)
- added G1: CoufalElektronika_logo, IMUnav:Coufal_elektronika_text_30x13mm, F.Cu at (112.4, 81.0)
- added G2: CoufalElektronika_logo, IMUnav:Coufal_elektronika_notext_10mm, F.Cu at (129.5, 91.5)
- added H1: MountingHole, MountingHole:MountingHole_3.2mm_M3, F.Cu at (93.0, 78.1)
- added H2: MountingHole, MountingHole:MountingHole_3.2mm_M3, F.Cu at (93.0, 86.0)
- added H3: MountingHole, MountingHole:MountingHole_3.2mm_M3, F.Cu at (93.0, 94.0)
- added H4: MountingHole, MountingHole:MountingHole_3.2mm_M3, F.Cu at (93.0, 102.0)
- added J1: Conn_01x03_Pin, Connector_PinHeader_2.54mm:PinHeader_1x03_P2.54mm_Vertical, F.Cu at (99.3, 89.2)
- added J2: Conn_01x03_Pin, Connector_PinHeader_2.54mm:PinHeader_1x03_P2.54mm_Vertical, F.Cu at (104.0, 89.2)
- added J3: Conn_01x03_Pin, Connector_PinHeader_2.54mm:PinHeader_1x03_P2.54mm_Vertical, F.Cu at (108.6, 89.2)
- added J4: Conn_01x03_Pin, Connector_PinHeader_2.54mm:PinHeader_1x03_P2.54mm_Vertical, F.Cu at (113.2, 89.2)
- added J5: Conn_01x03_Pin, Connector_PinHeader_2.54mm:PinHeader_1x03_P2.54mm_Vertical, F.Cu at (117.9, 89.2)
- added J6: Conn_01x03_Pin, Connector_PinHeader_2.54mm:PinHeader_1x03_P2.54mm_Vertical, F.Cu at (122.5, 89.2)
- added J7: 918-418K2023S40001, Connector_USB:USB_C_Receptacle_HRO_TYPE-C-31-M-12, F.Cu at (76.0, 61.2)
- added J8: Conn_Coaxial, Connector_Coaxial:SMA_Amphenol_901-143_Horizontal, F.Cu at (162.4, 86.7)
- added J9: Micro_SD_Card_Det_Hirose_DM3AT, Connector_Card:microSD_HC_Hirose_DM3AT-SF-PEJM5, F.Cu at (97.4, 126.4)
- added L1: 470n, Inductor_SMD:L_Chilisin_BMRA00040420, F.Cu at (97.1, 63.1)
- added Q1: S8050, Package_TO_SOT_SMD:SOT-23, F.Cu at (155.3, 120.2)
- added Q2: S8050, Package_TO_SOT_SMD:SOT-23, F.Cu at (155.3, 124.7)
- added R1: 10K, Resistor_SMD:R_0603_1608Metric, F.Cu at (130.1, 97.8)
- added R10: 10K, Resistor_SMD:R_0603_1608Metric, F.Cu at (134.2, 105.3)
- added R11: 10K, Resistor_SMD:R_0603_1608Metric, F.Cu at (134.2, 107.8)
- added R12: 10K, Resistor_SMD:R_0603_1608Metric, F.Cu at (134.2, 110.3)
- added R13: 100K, Resistor_SMD:R_0603_1608Metric, F.Cu at (55.1, 55.8)
- added R14: 100K, Resistor_SMD:R_0603_1608Metric, F.Cu at (55.1, 58.3)
- added R15: 100K, Resistor_SMD:R_0603_1608Metric, F.Cu at (55.1, 60.8)
- added R16: 10K, Resistor_SMD:R_0603_1608Metric, F.Cu at (55.1, 63.3)
- added R17: 10K, Resistor_SMD:R_0603_1608Metric, F.Cu at (55.1, 65.8)
- added R18: 1K8, Resistor_SMD:R_0603_1608Metric, F.Cu at (55.1, 68.4)
- added R19: 1K8, Resistor_SMD:R_0603_1608Metric, F.Cu at (55.1, 70.9)
- added R2: 10K, Resistor_SMD:R_0603_1608Metric, F.Cu at (130.1, 100.3)
- added R20: 27K, Resistor_SMD:R_0603_1608Metric, F.Cu at (59.1, 48.3)
- added R21: 33K, Resistor_SMD:R_0603_1608Metric, F.Cu at (59.1, 50.8)
- added R22: 1K8, Resistor_SMD:R_0603_1608Metric, F.Cu at (59.1, 53.3)
- added R23: 10K, Resistor_SMD:R_0603_1608Metric, F.Cu at (59.1, 55.8)
- added R24: 30K, Resistor_SMD:R_0603_1608Metric, F.Cu at (59.1, 58.3)
- added R25: 10K, Resistor_SMD:R_0603_1608Metric, F.Cu at (59.1, 60.8)
- added R26: 1K, Resistor_SMD:R_0603_1608Metric, F.Cu at (59.1, 63.3)
- added R27: 5K1, Resistor_SMD:R_0603_1608Metric, F.Cu at (59.1, 65.8)
- added R28: 5K1, Resistor_SMD:R_0603_1608Metric, F.Cu at (59.1, 68.4)
- added R29: 100K, Resistor_SMD:R_0603_1608Metric, F.Cu at (59.1, 70.9)
- added R3: 10K, Resistor_SMD:R_0603_1608Metric, F.Cu at (130.1, 102.8)
- added R30: 100K, Resistor_SMD:R_0603_1608Metric, F.Cu at (63.1, 48.3)
- added R31: 100K, Resistor_SMD:R_0603_1608Metric, F.Cu at (63.1, 50.8)
- added R32: 12K, Resistor_SMD:R_0603_1608Metric, F.Cu at (63.1, 53.3)
- added R33: 100K, Resistor_SMD:R_0603_1608Metric, F.Cu at (63.1, 55.8)
- added R34: 470R, Resistor_SMD:R_0603_1608Metric, F.Cu at (63.1, 58.3)
- added R35: 100K, Resistor_SMD:R_0603_1608Metric, F.Cu at (63.1, 60.8)
- added R36: 68K, Resistor_SMD:R_0603_1608Metric, F.Cu at (63.1, 63.3)
- added R37: 15K, Resistor_SMD:R_0603_1608Metric, F.Cu at (63.1, 65.8)
- added R38: 470R, Resistor_SMD:R_0603_1608Metric, F.Cu at (63.1, 68.4)
- added R39: 33R, Resistor_SMD:R_0603_1608Metric, F.Cu at (144.2, 118.9)
- added R4: 10K, Resistor_SMD:R_0603_1608Metric, F.Cu at (130.1, 105.3)
- added R40: 33R, Resistor_SMD:R_0603_1608Metric, F.Cu at (144.2, 121.4)
- added R41: 10K, Resistor_SMD:R_0603_1608Metric, F.Cu at (144.2, 123.9)
- added R42: 470R, Resistor_SMD:R_0603_1608Metric, F.Cu at (144.2, 126.4)
- added R43: 470R, Resistor_SMD:R_0603_1608Metric, F.Cu at (148.2, 118.9)
- added R44: 12K, Resistor_SMD:R_0603_1608Metric, F.Cu at (148.2, 121.4)
- added R45: 12K, Resistor_SMD:R_0603_1608Metric, F.Cu at (148.2, 123.9)
- added R46: 10K, Resistor_SMD:R_0603_1608Metric, F.Cu at (148.2, 126.4)
- added R47: 33R, Resistor_SMD:R_0603_1608Metric, F.Cu at (74.7, 117.3)
- added R48: 33R, Resistor_SMD:R_0603_1608Metric, F.Cu at (74.7, 119.8)
- added R49: 33R, Resistor_SMD:R_0603_1608Metric, F.Cu at (74.7, 122.3)
- added R5: 10K, Resistor_SMD:R_0603_1608Metric, F.Cu at (130.1, 107.8)
- added R50: 33R, Resistor_SMD:R_0603_1608Metric, F.Cu at (78.7, 109.8)
- added R51: 33R, Resistor_SMD:R_0603_1608Metric, F.Cu at (78.7, 112.3)
- added R52: 33R, Resistor_SMD:R_0603_1608Metric, F.Cu at (78.7, 114.8)
- added R53: 100K, Resistor_SMD:R_0603_1608Metric, F.Cu at (78.7, 117.3)
- added R54: 100K, Resistor_SMD:R_0603_1608Metric, F.Cu at (140.2, 85.4)
- added R55: 100K, Resistor_SMD:R_0603_1608Metric, F.Cu at (140.2, 87.9)
- added R56: 33R, Resistor_SMD:R_0603_1608Metric, F.Cu at (140.2, 90.4)
- added R57: 33R, Resistor_SMD:R_0603_1608Metric, F.Cu at (140.2, 93.0)
- added R58: 10R, Resistor_SMD:R_0603_1608Metric, F.Cu at (140.2, 95.5)
- added R59: 33R, Resistor_SMD:R_0603_1608Metric, F.Cu at (107.8, 125.8)
- added R6: 10K, Resistor_SMD:R_0603_1608Metric, F.Cu at (130.1, 110.3)
- added R60: 33R, Resistor_SMD:R_0603_1608Metric, F.Cu at (107.8, 128.3)
- added R61: 33R, Resistor_SMD:R_0603_1608Metric, F.Cu at (107.8, 130.8)
- added R62: 33R, Resistor_SMD:R_0603_1608Metric, F.Cu at (107.8, 133.3)
- added R63: 33R, Resistor_SMD:R_0603_1608Metric, F.Cu at (111.8, 118.3)
- added R64: 33R, Resistor_SMD:R_0603_1608Metric, F.Cu at (111.8, 120.8)
- added R65: 33R, Resistor_SMD:R_0603_1608Metric, F.Cu at (111.8, 123.3)
- added R66: 33R, Resistor_SMD:R_0603_1608Metric, F.Cu at (111.8, 125.8)
- added R67: 33R, Resistor_SMD:R_0603_1608Metric, F.Cu at (111.8, 128.3)
- added R68: 33R, Resistor_SMD:R_0603_1608Metric, F.Cu at (111.8, 130.8)
- added R69: 33R, Resistor_SMD:R_0603_1608Metric, F.Cu at (111.8, 133.3)
- added R7: 33R, Resistor_SMD:R_0603_1608Metric, F.Cu at (134.2, 97.8)
- added R70: 33R, Resistor_SMD:R_0603_1608Metric, F.Cu at (115.8, 118.3)
- added R71: 10K, Resistor_SMD:R_0603_1608Metric, F.Cu at (115.8, 120.8)
- added R72: 10K, Resistor_SMD:R_0603_1608Metric, F.Cu at (115.8, 123.3)
- added R73: 10K, Resistor_SMD:R_0603_1608Metric, F.Cu at (115.8, 125.8)
- added R74: 10K, Resistor_SMD:R_0603_1608Metric, F.Cu at (115.8, 128.3)
- added R75: 10K, Resistor_SMD:R_0603_1608Metric, F.Cu at (115.8, 130.8)
- added R76: 10K, Resistor_SMD:R_0603_1608Metric, F.Cu at (115.8, 133.3)
- added R77: 10K, Resistor_SMD:R_0603_1608Metric, F.Cu at (119.8, 118.3)
- added R78: 10K, Resistor_SMD:R_0603_1608Metric, F.Cu at (119.8, 120.8)
- added R79: 10K, Resistor_SMD:R_0603_1608Metric, F.Cu at (119.8, 123.3)
- added R8: 33R, Resistor_SMD:R_0603_1608Metric, F.Cu at (134.2, 100.3)
- added R80: 10K, Resistor_SMD:R_0603_1608Metric, F.Cu at (119.8, 125.8)
- added R81: 10K, Resistor_SMD:R_0603_1608Metric, F.Cu at (119.8, 128.3)
- added R82: 10K, Resistor_SMD:R_0603_1608Metric, F.Cu at (119.8, 130.8)
- added R83: 1K8, Resistor_SMD:R_0603_1608Metric, F.Cu at (167.6, 39.3)
- added R84: 1K8, Resistor_SMD:R_0603_1608Metric, F.Cu at (167.6, 41.8)
- added R85: 1K8, Resistor_SMD:R_0603_1608Metric, F.Cu at (167.6, 44.3)
- added R9: 10K, Resistor_SMD:R_0603_1608Metric, F.Cu at (134.2, 102.8)
- added RESET1: SW_SPST, Button_Switch_SMD:SW_SPST_TL3342, F.Cu at (157.7, 103.0)
- added SW1: MT-102, IMUnav:TE_A101SYCQ04, F.Cu at (78.1, 51.2)
- added SW2: SW_SPST, Button_Switch_THT:SW_PUSH_6mm_H13mm, F.Cu at (128.5, 27.5)
- added SW3: SW_SPST, Button_Switch_THT:SW_PUSH_6mm_H13mm, F.Cu at (128.5, 36.0)
- added SW4: SW_SPST, Button_Switch_THT:SW_PUSH_6mm_H13mm, F.Cu at (128.5, 44.6)
- added SW5: SW_SPST, Button_Switch_THT:SW_PUSH_6mm_H13mm, F.Cu at (128.5, 53.1)
- added SWD1: Conn_01x06_Pin, Connector_PinHeader_2.54mm:PinHeader_1x06_P2.54mm_Vertical, F.Cu at (117.8, 98.8)
- added TP1: TestPoint, TestPoint:TestPoint_Keystone_5005-5009_Compact, F.Cu at (67.6, 49.5)
- added TP2: TestPoint, TestPoint:TestPoint_Keystone_5005-5009_Compact, F.Cu at (67.6, 54.6)
- added TP3: TestPoint, TestPoint:TestPoint_Keystone_5005-5009_Compact, F.Cu at (67.6, 59.6)
- added TP4: TestPoint, TestPoint:TestPoint_Keystone_5005-5009_Compact, F.Cu at (67.6, 64.7)
- added U1: STM32F446VETx, Package_QFP:LQFP-100_14x14mm_P0.5mm, F.Cu at (106.2, 105.8)
- added U10: ESP32-C3-MINI-1, PCM_Espressif:ESP32-C3-MINI-1, F.Cu at (145.5, 108.6)
- added U11: MPU-6050, Sensor_Motion:InvenSense_QFN-24_4x4mm_P0.5mm, F.Cu at (83.8, 111.7)
- added U12: LSM303C, Package_LGA:LGA-12_2x2mm_P0.5mm, F.Cu at (82.5, 122.6)
- added U13: ADIS16505-2BMLZ, IMUnav:BGA-100_10x10_15.0x15.0mm, F.Cu at (56.4, 119.9)
- added U14: ADIS16505-x/PCBZ, IMUnav:ADIS16505-PCBZ, F.Cu at (55.1, 91.3)
- added U15: XC6206P332MR, Package_TO_SOT_SMD:SOT-23-3, F.Cu at (164.5, 93.7)
- added U16: NEO-M8U, RF_GPS:ublox_NEO, F.Cu at (149.8, 82.9)
- added U17: XT25F256BWSIGT, Package_SON:WSON-8-1EP_8x6mm_P1.27mm_EP3.4x4.3mm, F.Cu at (110.6, 138.4)
- added U18: OLED_I2C, IMUnav:Display_128x64_096_I2C, F.Cu at (151.3, 27.4)
- added U2: TVS0500DRV, Package_SON:WSON-6-1EP_2x2mm_P0.65mm_EP1x1.6mm, F.Cu at (103.8, 67.8)
- added U3: 74LVC2G02, Package_SO:VSSOP-8_2.3x2mm_P0.5mm, F.Cu at (104.7, 52.1)
- added U4: BQ24075RGT, Package_DFN_QFN:VQFN-16-1EP_3x3mm_P0.5mm_EP1.6x1.6mm, F.Cu at (104.6, 56.6)
- added U5: USBLC6-2P6, Package_TO_SOT_SMD:SOT-666, F.Cu at (104.0, 60.8)
- added U6: HT7533-1, Package_TO_SOT_SMD:SOT-89-3, F.Cu at (97.1, 69.0)
- added U7: TPS62823DLC, Package_DFN_QFN:Texas_VSON-HR-8_1.5x2mm_P0.5mm, F.Cu at (103.8, 64.2)
- added U8: USB2514B-AEZC-TR, Package_DFN_QFN:QFN-36-1EP_6x6mm_P0.5mm_EP3.7x3.7mm, F.Cu at (97.8, 51.1)
- added U9: CH340G, Package_SO:SOIC-16_3.9x9.9mm_P1.27mm, F.Cu at (157.1, 112.3)
- added X1: SX5M24.000M20F30TNN, IMUnav:OSC_ECS-3963-250-BN-TR, F.Cu at (131.3, 76.6)
- added X2: SX5M24.000M20F30TNN, IMUnav:OSC_ECS-3963-250-BN-TR, F.Cu at (97.4, 57.8)
