File: Hardware/IMUnav_H00/IMUnav_H00.kicad_pcb (KiCad board)
At the start: 4 copper layers, 100 x 100 mm, 220 parts, among them J1 Conn_ARM_JTAG_SWD_10, J2 Conn_01x03_Pin, J3 Conn_01x03_Pin, J4 Conn_01x03_Pin, J5 Conn_01x03_Pin, J6 Conn_01x03_Pin, J7 918-418K2023S40001, J8 SMA6252A2-3GT50G-50, J9 Micro_SD_Card_Det_Hirose_DM3AT, Q1 S8050, Q2 S8050, SW1 MT-102, SW2 SW_SPST, SW3 SW_SPST, SW4 SW_SPST, SW5 SW_SPST, U1 STM32F446VETx, U10 ESP32-C3-MINI-1, U11 MPU-6050, U12 LSM303AGR, U13 ADIS16505-2BMLZ, U14 ADIS16505-x/PCBZ, U15 XC6206P332MR, U16 NEO-M8U, U17 XT25F256BWSIGT, U18 OLED_I2C, U2 TVS0500DRV, U3 74LVC2G02, U4 BQ24075RGT, U5 USBLC6-2P6, U6 HT7533-1, U7 TPS62823DLC, U8 USB2514B-AEZC-TR, U9 CH340G, X1 SX5M24.000M20F30TNN, X2 SX5M24.000M20F30TNN

Commit message: PCB touch-ups, bom file for testing
Changed lines of the file:
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@@
     (property "ki_keywords" "R res resistor")
     (attr smd)
-    (fp_text reference "R2" (at 0 -1.43 90) (layer "F.SilkS")
+    (fp_text reference "R2" (at -0.508 -1.27 90) (layer "F.SilkS")
         (effects (font (size 1 1) (thickness 0.15)))
     )
@@
     (property "Sheetfile" "IMUnav_H00.kicad_sch")
     (property "Sheetname" "")
+    (property "exclude_from_bom" "")
     (property "ki_description" "Generic connector, single row, 01x03, script generated")
     (property "ki_keywords" "connector")
-    (attr through_hole)
+    (attr through_hole exclude_from_bom)
     (fp_text reference "J6" (at 2.286 -1.031 180) (layer "F.SilkS")
         (effects (font (size 1 1) (thickness 0.15)))
@@
     (property "ki_keywords" "cap capacitor")
     (attr smd)
-    (fp_text reference "C19" (at 0 -1.43) (layer "F.SilkS")
+    (fp_text reference "C19" (at 0 -1.651) (layer "F.SilkS")
         (effects (font (size 1 1) (thickness 0.15)))
     )
@@
     (property "ki_keywords" "cap capacitor")
     (attr smd)
-    (fp_text reference "C32" (at 2.667 0.254 90) (layer "F.SilkS")
+    (fp_text reference "C32" (at 2.667 0.508 90) (layer "F.SilkS")
         (effects (font (size 0.8 0.8) (thickness 0.15)))
     )
@@
     (property "Sheetfile" "IMUnav_H00.kicad_sch")
     (property "Sheetname" "")
+    (property "exclude_from_bom" "")
     (property "ki_description" "Generic connector, single row, 01x03, script generated")
     (property "ki_keywords" "connector")
-    (attr through_hole)
+    (attr through_hole exclude_from_bom)
     (fp_text reference "J5" (at -2.286 0.874 180) (layer "F.SilkS")
         (effects (font (size 1 1) (thickness 0.15)))
@@
     (property "Sheetfile" "IMUnav_H00.kicad_sch")
     (property "Sheetname" "")
+    (property "exclude_from_bom" "")
     (property "ki_description" "Generic connector, single row, 01x03, script generated")
     (property "ki_keywords" "connector")
-    (attr through_hole)
+    (attr through_hole exclude_from_bom)
     (fp_text reference "J3" (at 2.413 4.049 -180) (layer "F.SilkS")
         (effects (font (size 0.8 0.8) (thickness 0.15)))
@@
     (descr "Inductor, Chilisin, BMRA00040420, 4.6x4.1x2.0mm, https://www.chilisin.com/upload/media/product/power/file/BMRx_Series.pdf")
     (tags "Inductor bmrx mchi")
+    (property "LCSC" "C280580")
     (property "Sheetfile" "USB+Power.kicad_sch")
     (property "Sheetname" "USB+Power")
@@
     (property "ki_keywords" "cap capacitor")
     (attr smd)
-    (fp_text reference "C13" (at 0.324 1.328 90) (layer "F.SilkS")
+    (fp_text reference "C13" (at 0.451 1.328 90) (layer "F.SilkS")
         (effects (font (size 0.8 0.8) (thickness 0.15)))
     )
@@
     (property "ki_keywords" "BNC SMA SMB SMC LEMO coaxial connector CINCH RCA")
     (attr through_hole)
-    (fp_text reference "J8" (at -5.2 0 90) (layer "F.SilkS")
+    (fp_text reference "J8" (at -3.048 5.065 180) (layer "F.SilkS")
         (effects (font (size 1 1) (thickness 0.15)))
     )
@@
     (property "ki_keywords" "R res resistor")
     (attr smd)
-    (fp_text reference "R18" (at 0 1.016 -270) (layer "F.SilkS")
+    (fp_text reference "R18" (at -1.898 0.254 -180) (layer "F.SilkS")
         (effects (font (size 0.8 0.8) (thickness 0.15)))
     )
@@
     (property "ki_keywords" "Crystal Clock Oscillator")
     (attr smd)
-    (fp_text reference "X1" (at 3.429 0.381) (layer "F.SilkS")
-        (effects (font (size 0.481173 0.481173) (thickness 0.15)))
+    (fp_text reference "X1" (at 3.556 0.254) (layer "F.SilkS")
+        (effects (font (size 0.8 0.8) (thickness 0.15)))
     )
     (fp_text value "SX5M24.000M20F30TNN" (at 4.002267 2.414222) (layer "F.Fab")
@@
     (property "Sheetfile" "IMUnav_H00.kicad_sch")
     (property "Sheetname" "")
+    (property "exclude_from_bom" "")
     (property "ki_description" "Cortex Debug Connector, standard ARM Cortex-M SWD and JTAG interface")
     (property "ki_keywords" "Cortex Debug Connector ARM SWD JTAG")
-    (attr through_hole)
+    (attr through_hole exclude_from_bom)
     (fp_text reference "J1" (at 0.635 -1.695) (layer "F.SilkS")
         (effects (font (size 1 1) (thickness 0.15)))
@@
     (property "ki_keywords" "esp32-c3")
     (attr smd)
-    (fp_text reference "U10" (at 0 -9.5 90) (layer "F.SilkS")
+    (fp_text reference "U10" (at -1.143 9.304 270) (layer "F.SilkS")
         (effects (font (size 1 1) (thickness 0.15)))
     )
@@
     (property "ki_keywords" "R res resistor")
     (attr smd)
-    (fp_text reference "R71" (at -0.001 -4.572 90) (layer "F.SilkS")
+    (fp_text reference "R71" (at -2.033 -1.397 -180) (layer "F.SilkS")
         (effects (font (size 0.8 0.8) (thickness 0.15)))
     )
@@
     (property "Sheetfile" "IMUnav_H00.kicad_sch")
     (property "Sheetname" "")
+    (property "exclude_from_bom" "")
     (property "ki_description" "Generic connector, single row, 01x03, script generated")
     (property "ki_keywords" "connector")
-    (attr through_hole)
+    (attr through_hole exclude_from_bom)
     (fp_text reference "J4" (at 0 -2.33 90) (layer "F.SilkS")
         (effects (font (size 1 1) (thickness 0.15)))
@@
     (property "ki_keywords" "R res resistor")
     (attr smd)
-    (fp_text reference "R1" (at 0 -1.43 90) (layer "F.SilkS")
+    (fp_text reference "R1" (at -0.381 1.27 90) (layer "F.SilkS")
         (effects (font (size 1 1) (thickness 0.15)))
     )
@@
     (property "ki_keywords" "cap capacitor")
     (attr smd)
-    (fp_text reference "C30" (at 0 -1.43) (layer "F.SilkS")
+    (fp_text reference "C30" (at -0.096 1.185) (layer "F.SilkS")
         (effects (font (size 0.8 0.8) (thickness 0.15)))
     )
@@
     (property "Sheetfile" "IMUnav_H00.kicad_sch")
     (property "Sheetname" "")
+    (property "exclude_from_bom" "")
     (property "ki_description" "Generic connector, single row, 01x03, script generated")
     (property "ki_keywords" "connector")
-    (attr through_hole)
+    (attr through_hole exclude_from_bom)
     (fp_text reference "J2" (at -2.286 3.62 180) (layer "F.SilkS")
         (effects (font (size 1 1) (thickness 0.15)))
