File: Hardware/IMUnav_H00/ESP32.kicad_sch (KiCad schematic)
At the start: 18 parts, among them U10 ESP32-C3-MINI-1

Commit message: Thesis - added appendix
Other:
- note added: "ESP32 WiFi/BT interface"
- title: (none) -> IMUnav
Changed lines of the file:
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@@
 (kicad_sch (version 20230121) (generator eeschema)
   (paper "A4")
+  (title_block
+    (title "IMUnav")
+    (date "2023-12-21")
+    (rev "H00")
+    (comment 1 "Inertial navigation unit")
+  )
   (junction (at 120.65 90.17) (diameter 0) (color 0 0 0 0)
   )
@@
     (stroke (width 0) (type default))
   )
+  (text "ESP32\nWiFi/BT interface" (at 83.82 71.12 0)
+    (effects (font (size 2.54 2.54) (thickness 0.508) bold) (justify left bottom))
+  )
   (hierarchical_label "ESP_TX1" (shape input) (at 199.39 137.16 0) (fields_autoplaced)
