File: Hardware/IMUnav_H00/GPS.kicad_sch (KiCad schematic)
At the start: 15 parts, among them J8 SMA6252A2-3GT50G-50, U15 XC6206P332MR, U16 NEO-M8U

Commit message: Silkscreen layout
Parts:
- renumbered C59 to C56, C60 to C57
Changed lines of the file:
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@@
         )
         (path "/4c2dd95e-3649-4040-ab57-00df6d22e0b0/61a7e487-220c-46a1-aef5-176736fd02e1"
-          (reference "#PWR0202") (unit 1)
+          (reference "#PWR0198") (unit 1)
         )
       )
@@
         )
         (path "/4c2dd95e-3649-4040-ab57-00df6d22e0b0/61a7e487-220c-46a1-aef5-176736fd02e1"
-          (reference "#PWR0193") (unit 1)
+          (reference "#PWR0189") (unit 1)
         )
       )
@@
         )
         (path "/4c2dd95e-3649-4040-ab57-00df6d22e0b0/61a7e487-220c-46a1-aef5-176736fd02e1"
-          (reference "#PWR0196") (unit 1)
+          (reference "#PWR0192") (unit 1)
         )
       )
@@
         )
         (path "/4c2dd95e-3649-4040-ab57-00df6d22e0b0/61a7e487-220c-46a1-aef5-176736fd02e1"
-          (reference "C61") (unit 1)
+          (reference "C58") (unit 1)
         )
       )
@@
         )
         (path "/4c2dd95e-3649-4040-ab57-00df6d22e0b0/61a7e487-220c-46a1-aef5-176736fd02e1"
+          (reference "#PWR0187") (unit 1)
+        )
+      )
+      (project "PaLampa_MoBo_H01"
+        (path "/68867493-9f89-4388-916e-56f5ada0ac5c"
+          (reference "#PWR?") (unit 1)
+        )
+      )
+    )
+  )
+  (symbol (lib_id "power:+3V3") (at 151.13 50.8 0) (unit 1)
+    (in_bom yes) (on_board yes) (dnp no)
+    (property "Reference" "#PWR03" (at 151.13 54.61 0)
+      (effects (font (size 1.27 1.27)) hide)
+    )
+    (property "Value" "+3V3" (at 151.511 46.4058 0)
+      (effects (font (size 1.27 1.27)))
+    )
+    (property "Footprint" "" (at 151.13 50.8 0)
+      (effects (font (size 1.27 1.27)) hide)
+    )
+    (property "Datasheet" "" (at 151.13 50.8 0)
+      (effects (font (size 1.27 1.27)) hide)
+    )
+    (pin "1")
+    (instances
+      (project "IMUnav_H00"
+        (path "/4c2dd95e-3649-4040-ab57-00df6d22e0b0"
+          (reference "#PWR03") (unit 1)
+        )
+        (path "/4c2dd95e-3649-4040-ab57-00df6d22e0b0/61a7e487-220c-46a1-aef5-176736fd02e1"
           (reference "#PWR0191") (unit 1)
         )
@@
     )
   )
-  (symbol (lib_id "power:+3V3") (at 151.13 50.8 0) (unit 1)
-    (in_bom yes) (on_board yes) (dnp no)
-    (property "Reference" "#PWR03" (at 151.13 54.61 0)
-      (effects (font (size 1.27 1.27)) hide)
-    )
-    (property "Value" "+3V3" (at 151.511 46.4058 0)
-      (effects (font (size 1.27 1.27)))
-    )
-    (property "Footprint" "" (at 151.13 50.8 0)
-      (effects (font (size 1.27 1.27)) hide)
-    )
-    (property "Datasheet" "" (at 151.13 50.8 0)
-      (effects (font (size 1.27 1.27)) hide)
-    )
-    (pin "1")
-    (instances
-      (project "IMUnav_H00"
-        (path "/4c2dd95e-3649-4040-ab57-00df6d22e0b0"
-          (reference "#PWR03") (unit 1)
-        )
-        (path "/4c2dd95e-3649-4040-ab57-00df6d22e0b0/61a7e487-220c-46a1-aef5-176736fd02e1"
-          (reference "#PWR0195") (unit 1)
-        )
-      )
-      (project "PaLampa_MoBo_H01"
-        (path "/68867493-9f89-4388-916e-56f5ada0ac5c"
-          (reference "#PWR?") (unit 1)
-        )
-      )
-    )
-  )
   (symbol (lib_id "Device:C") (at 196.85 54.61 0) (unit 1)
     (in_bom yes) (on_board yes) (dnp no)
@@
         )
         (path "/4c2dd95e-3649-4040-ab57-00df6d22e0b0/61a7e487-220c-46a1-aef5-176736fd02e1"
-          (reference "C62") (unit 1)
+          (reference "C59") (unit 1)
         )
       )
@@
         )
         (path "/4c2dd95e-3649-4040-ab57-00df6d22e0b0/61a7e487-220c-46a1-aef5-176736fd02e1"
-          (reference "#PWR0192") (unit 1)
+          (reference "#PWR0188") (unit 1)
         )
       )
@@
         )
         (path "/4c2dd95e-3649-4040-ab57-00df6d22e0b0/61a7e487-220c-46a1-aef5-176736fd02e1"
-          (reference "#PWR0190") (unit 1)
+          (reference "#PWR0186") (unit 1)
         )
       )
@@
         )
         (path "/4c2dd95e-3649-4040-ab57-00df6d22e0b0/61a7e487-220c-46a1-aef5-176736fd02e1"
-          (reference "#PWR0189") (unit 1)
+          (reference "#PWR0185") (unit 1)
         )
       )
@@
   (symbol (lib_id "Device:C") (at 44.45 33.02 0) (unit 1)
     (in_bom yes) (on_board yes) (dnp no) (fields_autoplaced)
-    (property "Reference" "C59" (at 47.371 31.8079 0)
+    (property "Reference" "C56" (at 47.371 31.8079 0)
       (effects (font (size 1.27 1.27)) (justify left))
     )
@@
       (project "IMUnav_H00"
         (path "/4c2dd95e-3649-4040-ab57-00df6d22e0b0/61a7e487-220c-46a1-aef5-176736fd02e1"
-          (reference "C59") (unit 1)
+          (reference "C56") (unit 1)
         )
       )
@@
         )
         (path "/4c2dd95e-3649-4040-ab57-00df6d22e0b0/61a7e487-220c-46a1-aef5-176736fd02e1"
-          (reference "C64") (unit 1)
+          (reference "C61") (unit 1)
         )
       )
@@
         )
         (path "/4c2dd95e-3649-4040-ab57-00df6d22e0b0/61a7e487-220c-46a1-aef5-176736fd02e1"
-          (reference "#PWR0188") (unit 1)
+          (reference "#PWR0184") (unit 1)
         )
       )
@@
         )
         (path "/4c2dd95e-3649-4040-ab57-00df6d22e0b0/61a7e487-220c-46a1-aef5-176736fd02e1"
-          (reference "C63") (unit 1)
+          (reference "C60") (unit 1)
         )
       )
@@
         )
         (path "/4c2dd95e-3649-4040-ab57-00df6d22e0b0/61a7e487-220c-46a1-aef5-176736fd02e1"
-          (reference "#PWR0198") (unit 1)
+          (reference "#PWR0194") (unit 1)
         )
       )
@@
   (symbol (lib_id "Device:C") (at 77.47 33.02 0) (unit 1)
     (in_bom yes) (on_board yes) (dnp no) (fields_autoplaced)
-    (property "Reference" "C60" (at 80.391 31.8079 0)
+    (property "Reference" "C57" (at 80.391 31.8079 0)
       (effects (font (size 1.27 1.27)) (justify left))
     )
@@
       (project "IMUnav_H00"
         (path "/4c2dd95e-3649-4040-ab57-00df6d22e0b0/61a7e487-220c-46a1-aef5-176736fd02e1"
-          (reference "C60") (unit 1)
+          (reference "C57") (unit 1)
         )
       )
@@
         )
         (path "/4c2dd95e-3649-4040-ab57-00df6d22e0b0/61a7e487-220c-46a1-aef5-176736fd02e1"
-          (reference "#PWR0199") (unit 1)
+          (reference "#PWR0195") (unit 1)
         )
       )
@@
         )
         (path "/4c2dd95e-3649-4040-ab57-00df6d22e0b0/61a7e487-220c-46a1-aef5-176736fd02e1"
-          (reference "#PWR0197") (unit 1)
+          (reference "#PWR0193") (unit 1)
         )
       )
@@
         )
         (path "/4c2dd95e-3649-4040-ab57-00df6d22e0b0/61a7e487-220c-46a1-aef5-176736fd02e1"
-          (reference "#PWR0187") (unit 1)
+          (reference "#PWR0183") (unit 1)
         )
       )
@@
         )
         (path "/4c2dd95e-3649-4040-ab57-00df6d22e0b0/61a7e487-220c-46a1-aef5-176736fd02e1"
-          (reference "#PWR0201") (unit 1)
+          (reference "#PWR0197") (unit 1)
         )
       )
@@
         )
         (path "/4c2dd95e-3649-4040-ab57-00df6d22e0b0/61a7e487-220c-46a1-aef5-176736fd02e1"
-          (reference "#PWR0200") (unit 1)
+          (reference "#PWR0196") (unit 1)
         )
       )
@@
         )
         (path "/4c2dd95e-3649-4040-ab57-00df6d22e0b0/61a7e487-220c-46a1-aef5-176736fd02e1"
-          (reference "#PWR0194") (unit 1)
-        )
-      )
+          (reference "#PWR0190") (unit 1)
+        )
+      )

Commit message: Thesis - added appendix
Other:
- note added: "GPS module + external antenna"
- title: (none) -> IMUnav
- moved on the sheet: C1, C2, C56, C57, FB3, J8, R10, R30, R58, U15, U16
