File: Hardware/IMUnav_H00/Memory.kicad_sch (KiCad schematic)
At the start: 29 parts, among them J3 Micro_SD_Card_Det_Hirose_DM3AT, U2 XT25F256BWSIGT

Commit message: Changed LSM303C to LSM303AGR
Connections:
- net GND: now also J3.11 (SHIELD)
Changed lines of the file:
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@@
+    )
+  )
+  (symbol (lib_id "power:GND") (at 185.42 69.85 0) (unit 1)
+    (in_bom yes) (on_board yes) (dnp no)
+    (property "Reference" "#PWR04" (at 185.42 76.2 0)
+      (effects (font (size 1.27 1.27)) hide)
+    )
+    (property "Value" "GND" (at 185.547 74.2442 0)
+      (effects (font (size 1.27 1.27)))
+    )
+    (property "Footprint" "" (at 185.42 69.85 0)
+      (effects (font (size 1.27 1.27)) hide)
+    )
+    (property "Datasheet" "" (at 185.42 69.85 0)
+      (effects (font (size 1.27 1.27)) hide)
+    )
+    (pin "1")
+    (instances
+      (project "IMUnav_H00"
+        (path "/4c2dd95e-3649-4040-ab57-00df6d22e0b0"
+          (reference "#PWR04") (unit 1)
+        )
+        (path "/4c2dd95e-3649-4040-ab57-00df6d22e0b0/86346d6f-e2e9-4b09-829f-5c51f1c26d9b"
+          (reference "#PWR0241") (unit 1)
+        )
+      )
+      (project "PaLampa_MoBo_H01"
+        (path "/68867493-9f89-4388-916e-56f5ada0ac5c"
+          (reference "#PWR?") (unit 1)
+        )
+      )
     )
   )

Commit message: Semi-final PCB routing (copper only)
Parts:
- added C?: 10u, Capacitor_SMD:C_0805_2012Metric, symbol Device:C
- R41: now not fitted
Connections:
- net +3V3: now also C?.1
- net GND: now also C?.2
Changed lines of the file:
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@@
+    (stroke (width 0) (type default))
+  )
+  (wire (pts (xy 194.31 132.08) (xy 194.31 139.7))
     (stroke (width 0) (type default))
   )
@@
   )
   (wire (pts (xy 132.08 119.38) (xy 137.16 119.38))
+    (stroke (width 0) (type default))
+  )
+  (wire (pts (xy 194.31 114.3) (xy 194.31 124.46))
     (stroke (width 0) (type default))
   )
@@
     )
   )
+  (symbol (lib_id "power:+3V3") (at 194.31 114.3 0) (unit 1)
+    (in_bom yes) (on_board yes) (dnp no)
+    (property "Reference" "#PWR03" (at 194.31 118.11 0)
+      (effects (font (size 1.27 1.27)) hide)
+    )
+    (property "Value" "+3V3" (at 194.691 109.9058 0)
+      (effects (font (size 1.27 1.27)))
+    )
+    (property "Footprint" "" (at 194.31 114.3 0)
+      (effects (font (size 1.27 1.27)) hide)
+    )
+    (property "Datasheet" "" (at 194.31 114.3 0)
+      (effects (font (size 1.27 1.27)) hide)
+    )
+    (pin "1")
+    (instances
+      (project "IMUnav_H00"
+        (path "/4c2dd95e-3649-4040-ab57-00df6d22e0b0"
+          (reference "#PWR03") (unit 1)
+        )
+        (path "/4c2dd95e-3649-4040-ab57-00df6d22e0b0/86346d6f-e2e9-4b09-829f-5c51f1c26d9b"
+          (reference "#PWR0181") (unit 1)
+        )
+      )
+      (project "PaLampa_MoBo_H01"
+        (path "/68867493-9f89-4388-916e-56f5ada0ac5c"
+          (reference "#PWR?") (unit 1)
+        )
+      )
+    )
+  )
   (symbol (lib_id "power:+3V3") (at 121.92 97.79 0) (unit 1)
     (in_bom yes) (on_board yes) (dnp no)
@@
         (path "/4c2dd95e-3649-4040-ab57-00df6d22e0b0/86346d6f-e2e9-4b09-829f-5c51f1c26d9b"
           (reference "#PWR0217") (unit 1)
+        )
+      )
+      (project "PaLampa_MoBo_H01"
+        (path "/68867493-9f89-4388-916e-56f5ada0ac5c"
+          (reference "#PWR?") (unit 1)
+        )
+      )
+    )
+  )
+  (symbol (lib_id "power:GND") (at 194.31 139.7 0) (unit 1)
+    (in_bom yes) (on_board yes) (dnp no)
+    (property "Reference" "#PWR04" (at 194.31 146.05 0)
+      (effects (font (size 1.27 1.27)) hide)
+    )
+    (property "Value" "GND" (at 194.437 144.0942 0)
+      (effects (font (size 1.27 1.27)))
+    )
+    (property "Footprint" "" (at 194.31 139.7 0)
+      (effects (font (size 1.27 1.27)) hide)
+    )
+    (property "Datasheet" "" (at 194.31 139.7 0)
+      (effects (font (size 1.27 1.27)) hide)
+    )
+    (pin "1")
+    (instances
+      (project "IMUnav_H00"
+        (path "/4c2dd95e-3649-4040-ab57-00df6d22e0b0"
+          (reference "#PWR04") (unit 1)
+        )
+        (path "/4c2dd95e-3649-4040-ab57-00df6d22e0b0/86346d6f-e2e9-4b09-829f-5c51f1c26d9b"
+          (reference "#PWR027") (unit 1)
         )
       )
@@
     )
   )
+  (symbol (lib_id "Device:C") (at 194.31 128.27 0) (unit 1)
+    (in_bom yes) (on_board yes) (dnp no)
+    (property "Reference" "C?" (at 197.231 127.1016 0)
+      (effects (font (size 1.27 1.27)) (justify left))
+    )
+    (property "Value" "10u" (at 197.231 129.413 0)
+      (effects (font (size 1.27 1.27)) (justify left))
+    )
+    (property "Footprint" "Capacitor_SMD:C_0805_2012Metric" (at 195.2752 132.08 0)
+      (effects (font (size 1.27 1.27)) hide)
+    )
+    (property "Datasheet" "~" (at 194.31 128.27 0)
+      (effects (font (size 1.27 1.27)) hide)
+    )
+    (property "LCSC" "C15850" (at 194.31 128.27 0)
+      (effects (font (size 1.27 1.27)) hide)
+    )
+    (pin "1")
+    (pin "2")
+    (instances
+      (project "IMUnav_H00"
+        (path "/4c2dd95e-3649-4040-ab57-00df6d22e0b0/6fbc37c5-87b4-45e0-ab4e-6fb233c6fd9b"
+          (reference "C?") (unit 1)
+        )
+        (path "/4c2dd95e-3649-4040-ab57-00df6d22e0b0/bf35eb2a-37f7-4f5f-b34e-af3028cdd96b"
+          (reference "C37") (unit 1)
+        )
+        (path "/4c2dd95e-3649-4040-ab57-00df6d22e0b0/86346d6f-e2e9-4b09-829f-5c51f1c26d9b"
+          (reference "C54") (unit 1)
+        )
+      )
+      (project "PaLampa_MoBo_H01"
+        (path "/68867493-9f89-4388-916e-56f5ada0ac5c/4ec8e228-d742-4cd8-8c0d-36879b06f45c"
+          (reference "C?") (unit 1)
+        )
+      )
+    )
+  )
   (symbol (lib_id "Device:R") (at 90.17 46.99 90) (unit 1)
     (in_bom yes) (on_board yes) (dnp no)
@@
   )
   (symbol (lib_id "Device:R") (at 116.84 30.48 0) (unit 1)
-    (in_bom yes) (on_board yes) (dnp no)
+    (in_bom yes) (on_board yes) (dnp yes)
     (property "Reference" "R41" (at 119.38 29.21 90)
       (effects (font (size 1.27 1.27)) (justify left))

Commit message: Thesis - added appendix
Other:
- note added: "External FLASH"
- note added: "microSD card"
- title: (none) -> IMUnav
Changed lines of the file:
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@@
 (kicad_sch (version 20230121) (generator eeschema)
   (paper "A4")
+  (title_block
+    (title "IMUnav")
+    (date "2023-12-21")
+    (rev "H00")
+    (comment 1 "Inertial navigation unit")
+  )
   (junction (at 116.84 57.15) (diameter 0) (color 0 0 0 0)
   )
@@
     (stroke (width 0) (type default))
   )
+  (text "External FLASH" (at 139.7 105.41 0)
+    (effects (font (size 2.54 2.54) (thickness 0.508) bold) (justify left bottom))
+  )
+  (text "microSD card" (at 152.4 27.94 0)
+    (effects (font (size 2.54 2.54) (thickness 0.508) bold) (justify left bottom))
+  )
   (hierarchical_label "QSPI_IO2" (shape input) (at 81.28 129.54 180) (fields_autoplaced)
