File: Hardware/IMUnav_H00/USB+Power.kicad_sch (KiCad schematic)
At the start: 74 parts, among them J7 918-418K2023S40001, SW1 MT-102, U1 USB2514B-AEZC-TR, U14 HT7533-1, U2 TVS0500DRV, U3 74LVC2G02, U4 BQ24075RGT, U5 USBLC6-2P6, U7 TPS62823DLC, X2 SX5M24.000M20F30TNN

Commit message: PCB routing
Parts:
- removed TP1: TestPoint, TestPoint:TestPoint_Keystone_5005-5009_Compact, symbol Connector:TestPoint
- TP2, TP3, TP4: footprint TestPoint:TestPoint_Keystone_5005-5009_Compact -> TestPoint:TestPoint_THTPad_D1.5mm_Drill0.7mm
Connections:
- net +BATT: now also SW1.2 (B); no longer SW1.1 (A)
- net at C16.1, TP4.1, U4.10 (OUT)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: now also SW1.1 (A); no longer SW1.2 (B)
Other:
- moved on the sheet: SW1
Changed lines of the file:
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@@
   (junction (at 22.86 165.1) (diameter 0) (color 0 0 0 0)
   )
-  (junction (at 66.04 162.56) (diameter 0) (color 0 0 0 0)
-  )
   (junction (at 99.06 62.23) (diameter 0) (color 0 0 0 0)
   )
@@
   (junction (at 168.91 81.28) (diameter 0) (color 0 0 0 0)
   )
+  (junction (at 99.06 152.4) (diameter 0) (color 0 0 0 0)
+  )
   (junction (at 167.64 20.32) (diameter 0) (color 0 0 0 0)
   )
@@
   (junction (at 264.16 20.32) (diameter 0) (color 0 0 0 0)
   )
-  (junction (at 99.06 152.4) (diameter 0) (color 0 0 0 0)
-  )
   (junction (at 63.5 162.56) (diameter 0) (color 0 0 0 0)
   )
@@
   )
   (no_connect (at 259.08 76.2))
-  (no_connect (at 101.6 135.89))
+  (no_connect (at 93.98 148.59))
   (no_connect (at 99.06 72.39))
   (no_connect (at 99.06 69.85))
@@
     (stroke (width 0) (type default))
   )
-  (wire (pts (xy 63.5 162.56) (xy 66.04 162.56))
+  (wire (pts (xy 63.5 162.56) (xy 69.85 162.56))
     (stroke (width 0) (type default))
   )
@@
     (stroke (width 0) (type default))
   )
+  (wire (pts (xy 99.06 148.59) (xy 99.06 152.4))
+    (stroke (width 0) (type default))
+  )
   (wire (pts (xy 68.58 180.34) (xy 68.58 182.88))
     (stroke (width 0) (type default))
@@
   )
   (wire (pts (xy 95.25 190.5) (xy 105.41 190.5))
+    (stroke (width 0) (type default))
+  )
+  (wire (pts (xy 96.52 134.62) (xy 96.52 138.43))
     (stroke (width 0) (type default))
   )
@@
     (stroke (width 0) (type default))
   )
-  (wire (pts (xy 99.06 146.05) (xy 99.06 152.4))
-    (stroke (width 0) (type default))
-  )
   (wire (pts (xy 222.25 134.62) (xy 229.87 134.62))
     (stroke (width 0) (type default))
@@
     (stroke (width 0) (type default))
   )
-  (wire (pts (xy 66.04 162.56) (xy 69.85 162.56))
-    (stroke (width 0) (type default))
-  )
   (wire (pts (xy 36.83 184.15) (xy 36.83 187.96))
     (stroke (width 0) (type default))
@@
   )
   (wire (pts (xy 222.25 143.51) (xy 222.25 144.78))
-    (stroke (width 0) (type default))
-  )
-  (wire (pts (xy 66.04 158.75) (xy 66.04 162.56))
     (stroke (width 0) (type default))
   )
@@
       (effects (font (size 1.27 1.27)) (justify left))
     )
-    (property "Footprint" "TestPoint:TestPoint_Keystone_5005-5009_Compact" (at 107.95 152.4 0)
+    (property "Footprint" "TestPoint:TestPoint_THTPad_D1.5mm_Drill0.7mm" (at 107.95 152.4 0)
       (effects (font (size 1.27 1.27)) hide)
     )
@@
     )
   )
-  (symbol (lib_id "power:+BATT") (at 96.52 135.89 0) (unit 1)
-    (in_bom yes) (on_board yes) (dnp no)
-    (property "Reference" "#PWR073" (at 96.52 139.7 0)
-      (effects (font (size 1.27 1.27)) hide)
-    )
-    (property "Value" "+BATT" (at 96.901 131.4958 0)
-      (effects (font (size 1.27 1.27)))
-    )
-    (property "Footprint" "" (at 96.52 135.89 0)
-      (effects (font (size 1.27 1.27)) hide)
-    )
-    (property "Datasheet" "" (at 96.52 135.89 0)
+  (symbol (lib_id "power:+BATT") (at 96.52 134.62 0) (unit 1)
+    (in_bom yes) (on_board yes) (dnp no)
+    (property "Reference" "#PWR073" (at 96.52 138.43 0)
+      (effects (font (size 1.27 1.27)) hide)
+    )
+    (property "Value" "+BATT" (at 96.901 130.2258 0)
+      (effects (font (size 1.27 1.27)))
+    )
+    (property "Footprint" "" (at 96.52 134.62 0)
+      (effects (font (size 1.27 1.27)) hide)
+    )
+    (property "Datasheet" "" (at 96.52 134.62 0)
       (effects (font (size 1.27 1.27)) hide)
     )
@@
     )
   )
-  (symbol (lib_id "Switch:SW_SPDT") (at 99.06 140.97 90) (unit 1)
-    (in_bom yes) (on_board yes) (dnp no)
-    (property "Reference" "SW1" (at 103.8352 139.8016 90)
+  (symbol (lib_id "Switch:SW_SPDT") (at 96.52 143.51 270) (unit 1)
+    (in_bom yes) (on_board yes) (dnp no)
+    (property "Reference" "SW1" (at 91.7448 144.6784 90)
       (effects (font (size 1.27 1.27)) (justify right))
     )
-    (property "Value" "MT-102" (at 103.8352 142.113 90)
+    (property "Value" "MT-102" (at 91.7448 142.367 90)
       (effects (font (size 1.27 1.27)) (justify right))
     )
-    (property "Footprint" "IMUnav:TE_A101SYCQ04" (at 99.06 140.97 0)
-      (effects (font (size 1.27 1.27)) hide)
-    )
-    (property "Datasheet" "~" (at 99.06 140.97 0)
+    (property "Footprint" "IMUnav:TE_A101SYCQ04" (at 96.52 143.51 0)
+      (effects (font (size 1.27 1.27)) hide)
+    )
+    (property "Datasheet" "~" (at 96.52 143.51 0)
       (effects (font (size 1.27 1.27)) hide)
     )
@@
       (effects (font (size 1.27 1.27)) (justify left))
     )
-    (property "Footprint" "TestPoint:TestPoint_Keystone_5005-5009_Compact" (at 279.4 134.62 0)
+    (property "Footprint" "TestPoint:TestPoint_THTPad_D1.5mm_Drill0.7mm" (at 279.4 134.62 0)
       (effects (font (size 1.27 1.27)) hide)
     )
@@
         (path "/68867493-9f89-4388-916e-56f5ada0ac5c/4ec8e228-d742-4cd8-8c0d-36879b06f45c"
           (reference "#PWR?") (unit 1)
-        )
-      )
-    )
-  )
-  (symbol (lib_id "Connector:TestPoint") (at 66.04 158.75 0) (unit 1)
-    (in_bom yes) (on_board yes) (dnp no) (fields_autoplaced)
-    (property "Reference" "TP1" (at 67.437 154.2359 0)
-      (effects (font (size 1.27 1.27)) (justify left))
-    )
-    (property "Value" "TestPoint" (at 67.437 156.6601 0)
-      (effects (font (size 1.27 1.27)) (justify left))
-    )
-    (property "Footprint" "TestPoint:TestPoint_Keystone_5005-5009_Compact" (at 71.12 158.75 0)
-      (effects (font (size 1.27 1.27)) hide)
-    )
-    (property "Datasheet" "~" (at 71.12 158.75 0)
-      (effects (font (size 1.27 1.27)) hide)
-    )
-    (pin "1")
-    (instances
-      (project "IMUnav_H00"
-        (path "/4c2dd95e-3649-4040-ab57-00df6d22e0b0/6fbc37c5-87b4-45e0-ab4e-6fb233c6fd9b"
-          (reference "TP1") (unit 1)
         )
       )
@@
       (effects (font (size 1.27 1.27)) (justify left))
     )
-    (property "Footprint" "TestPoint:TestPoint_Keystone_5005-5009_Compact" (at 130.81 120.65 0)
-      (effects (font (size 1.27 1.27)) hide)
-    )
+    (property "Footprint" "TestPoint:TestPoint_THTPad_D1.5mm_Drill0.7mm" (at 130.81 120.65 0)
+      (effects (font (size 1.27 1.27)) hide)
+    )

Commit message: Silkscreen layout
Parts:
- added TP5: TestPoint, TestPoint:TestPoint_THTPad_D1.5mm_Drill0.7mm, symbol Connector:TestPoint
- renumbered TP4 to TP1
Connections:
- net GND: now also TP5.1
Other:
- moved on the sheet: TP2

Commit message: PCB touch-ups, bom file for testing
Parts:
- L1: LCSC (none) -> C280580
Changed lines of the file:
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@@
+      (effects (font (size 1.27 1.27)) hide)
+    )
+    (property "LCSC" "C280580" (at 204.47 134.62 90)
       (effects (font (size 1.27 1.27)) hide)
     )

Commit message: Thesis - added appendix
Other:
- note added: "Battery to +3V3 DC/DC converter"
- note added: "USB + battery voltage sensing"
- note added: "USB + hub"
- note added: "battery charging SW disconnect"
- title: (none) -> IMUnav
Changed lines of the file:
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@@
 (kicad_sch (version 20230121) (generator eeschema)
   (paper "A4")
+  (title_block
+    (title "IMUnav")
+    (date "2023-12-21")
+    (rev "H00")
+    (comment 1 "Inertial navigation unit")
+  )
   (junction (at 157.48 170.18) (diameter 0) (color 0 0 0 0)
   )
@@
     (effects (font (size 1.27 1.27) bold) (justify left bottom))
   )
+  (text "USB + battery\nvoltage sensing" (at 24.13 114.3 0)
+    (effects (font (size 2.54 2.54) (thickness 0.508) bold) (justify left bottom))
+  )
   (text "R\n" (at 35.56 137.16 0)
     (effects (font (size 1.27 1.27)) (justify left bottom))
   )
+  (text "battery charging \nSW disconnect" (at 60.96 137.16 0)
+    (effects (font (size 2.54 2.54) (thickness 0.508) bold) (justify left bottom))
+  )
+  (text "Battery to +3V3 DC/DC converter" (at 168.91 123.19 0)
+    (effects (font (size 2.54 2.54) (thickness 0.508) bold) (justify left bottom))
+  )
   (text "S" (at 35.56 168.91 0)
     (effects (font (size 1.27 1.27)) (justify left bottom))
   )
+  (text "USB + hub" (at 54.61 31.75 0)
+    (effects (font (size 2.54 2.54) (thickness 0.508) bold) (justify left bottom))
+  )
   (text "~{Q}" (at 64.77 166.37 0)
